Commit message: Degisikler falan fiso

File: youbot_description-kinetic-devel/robots/youbot.urdf.xacro (robot description, xacro)
@@ -22,4 +22,7 @@
   <!-- sensors -->
   <xacro:include filename="$(find youbot_description)/urdf/sensors/hokuyo_urg04_laser.urdf.xacro"/>
+  <xacro:include filename="$(find youbot_description)/urdf/sensors/asus_xtion_camera.urdf.xacro"/>
+   <!-- sensor tower -->
+  <xacro:include filename="$(find youbot_description)/urdf/misc/camera_tower.urdf.xacro"/>
   <!-- Now we can start using the macros xacro:included above to define the actual youbot -->
   <!-- The first use of a macro.  This one was defined in base.urdf.xacro above.
@@ -35,10 +38,12 @@
     <origin xyz="-0.159 0 0.046" rpy="0 0 0" />
   </xacro:youbot_plate>
-  <xacro:youbot_arm name="arm" parent="base_link">
-    <origin xyz="0.143 0 0.046" rpy="0 0 0" />
-  </xacro:youbot_arm>
-  <xacro:youbot_gripper name="gripper" parent="arm_link_5">
-    <origin xyz="0 0 0" rpy="0 0 0" />
-  </xacro:youbot_gripper>
+    <!-- camera tower -->
+  <xacro:camera_tower name="camera_tower" parent="plate_link">
+    <origin xyz="-0.11 0.0 0.03" rpy="0 0 0" />
+  </xacro:camera_tower>
+  <!-- 3D camera on tower -->
+  <xacro:asus_xtion_camera name="tower_cam3d" parent="camera_tower_link" tilt="0.0">
+    <origin xyz="0 0 0.49" rpy="0 0 0" />
+  </xacro:asus_xtion_camera>
   <!-- base laser front -->
   <xacro:hokuyo_urg04_laser name="base_laser_front" parent="base" ros_topic="scan_front" update_rate="10" min_angle="-1.57" max_angle="1.57">

File: youbot_description-kinetic-devel/urdf/youbot_base/base.gazebo.xacro (robot description, xacro)
@@ -11,6 +11,12 @@
       <kp>1000000</kp>
       <kd>100</kd>
+      <!-- Sürtünme parametreleri -->
+      <mu1>2.0</mu1>
+      <mu2>2.0</mu2>
     </gazebo>
     <gazebo reference="caster_link_fl">
+      <!-- Caster bağlantısı da yere temas ediyorsa, sürtünme eklenebilir -->
+      <mu1>2.0</mu1>
+      <mu2>2.0</mu2>
     </gazebo>
     <!-- front right wheel -->
@@ -18,6 +24,10 @@
       <kp>1000000</kp>
       <kd>100</kd>
+      <mu1>2.0</mu1>
+      <mu2>2.0</mu2>
     </gazebo>
     <gazebo reference="caster_link_fr">
+      <mu1>2.0</mu1>
+      <mu2>2.0</mu2>
     </gazebo>
     <!-- back left wheel -->
@@ -25,6 +35,10 @@
       <kp>1000000</kp>
       <kd>100</kd>
+      <mu1>2.0</mu1>
+      <mu2>2.0</mu2>
     </gazebo>
     <gazebo reference="caster_link_bl">
+      <mu1>2.0</mu1>
+      <mu2>2.0</mu2>
     </gazebo>
     <!-- back right wheel -->
@@ -32,6 +46,10 @@
       <kp>1000000</kp>
       <kd>100</kd>
+      <mu1>2.0</mu1>
+      <mu2>2.0</mu2>
     </gazebo>
     <gazebo reference="caster_link_br">
+      <mu1>2.0</mu1>
+      <mu2>2.0</mu2>
     </gazebo>
   </xacro:macro>

Commit message: son hali

File: youbot_description-kinetic-devel/robots/youbot.urdf.xacro (robot description, xacro)
@@ -35,4 +35,11 @@
   <!-- foot for arm-->
   <xacro:youbot_base name="base"/>
+  <xacro:youbot_arm name="arm" parent="base_link">
+    <!--<origin xyz="0.143 0 0.046" rpy="0 0 0" />-->
+    <origin xyz="0.123 0 0.046" rpy="0 0 0" /> <!-- x offset needs to be further verified -->
+  </xacro:youbot_arm>
+  <xacro:youbot_gripper name="gripper" parent="arm_link_5">
+    <origin xyz="0 0 0" rpy="0 0 0" />
+  </xacro:youbot_gripper>
   <xacro:youbot_plate name="plate" parent="base_link">
     <origin xyz="-0.159 0 0.046" rpy="0 0 0" />
